File: KICAD/untitled.kicad_sch (KiCad schematic)
At the start: 73 parts, among them IC1 TPA3116D2QDADRQ1, IC2 TPA3116D2QDADRQ1

Commit message: Ajout footprint
Parts:
- IC1, IC2: footprint SOP65P810X120-33N -> TPA3116D2QDADRQ1:SOP65P810X120-33N
Changed lines of the file:
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@@
 			)
 		)
-		(property "Footprint" "SOP65P810X120-33N"
+		(property "Footprint" "TPA3116D2QDADRQ1:SOP65P810X120-33N"
 			(at 177.8 157.15 0)
 			(effects
@@
 			)
 		)
-		(property "Footprint" "SOP65P810X120-33N"
+		(property "Footprint" "TPA3116D2QDADRQ1:SOP65P810X120-33N"
 			(at 177.8 244.78 0)
 			(effects
