File: KICAD/ADC.kicad_sch (KiCad schematic)
At the start: 5 parts, among them IC3 PCM1808PW

Commit message: clear
Parts:
- IC3: footprint Package_SO:TSSOP-14_4.4x5mm_P0.65mm -> footprints:PCM1808PW
Changed lines of the file:
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@@
 			)
 		)
-		(property "Footprint" "Package_SO:TSSOP-14_4.4x5mm_P0.65mm"
+		(property "Footprint" "footprints:PCM1808PW"
 			(at 148.59 187.63 0)
 			(hide yes)

Commit message: presque rien
Parts:
- removed C33, C35: 1u, symbol Device:C_Small
- removed C50: 100n, symbol Device:C_Small
- removed C53: 10u, symbol Device:C_Small
Connections:
- net +3.3V: no longer names the net of IC3.4 (VDD)
- net +5V: no longer names the net of IC3.3 (VCC)
- net BCK/SAI1_SCK_A: no longer names the net of IC3.8 (BCK)
- net DOUT/SAI1_SD_A: no longer names the net of IC3.9 (DOUT)
- removed net GND: IC3.10 (MD0), IC3.11 (MD1), IC3.12 (FMT), IC3.2 (AGND), IC3.5 (DGND)
- net LRCK/SAI1_FS_A: no longer names the net of IC3.7 (LRCK)
- net SCKI/SAI1_MCLK_A: no longer names the net of IC3.6 (SCKI)
