File: KICAD/DAC.kicad_sch (KiCad schematic)
At the start: 34 parts, among them IC4 PCM5102AQPWRQ1, IC6 PCM5102AQPWRQ1

Commit message: presque rien
Parts:
- removed C54, C57, C60, C64, C70, C71, C73, C75: 0,1u, symbol Device:C_Small
- removed C58, C59, C61, C65, C68, C69, C76, C77: 10u, symbol Device:C_Polarized_Small_US
- removed C62, C63, C72, C74, C80, C81: 2,2u, symbol Device:C_Small
- removed C66, C67, C78, C79: 2,2n, symbol Device:C_Small
- removed R18, R19, R20, R21: 470, symbol Device:R_Small
- removed R22, R23: 10k, symbol Device:R_Small
Connections:
- net +3.3V: no longer names the net of IC4.20 (DVDD)
- net +3.3V: no longer IC6.20 (DVDD)
- removed net +3.3VA: IC4.1 (CPVDD), IC4.8 (AVDD), IC6.1 (CPVDD), IC6.8 (AVDD)
- net BCKA: no longer names the net of IC6.13 (BCK)
- net BCKB: no longer names the net of IC4.13 (BCK)
- net DIN/SAI1_SD_A: no longer names the net of IC6.14 (DIN)
- net DIN/SAI1_SD_B: no longer names the net of IC4.14 (DIN)
- removed net GND: IC4.10 (DEMP), IC4.11 (FLT), IC4.12 (SCK), IC4.16 (FMT), IC4.19 (DGND), IC4.3 (CPGND), IC4.9 (AGND), IC6.10 (DEMP), IC6.11 (FLT), IC6.16 (FMT), IC6.19 (DGND), IC6.3 (CPGND), IC6.9 (AGND)
- net LRCKA: no longer names the net of IC6.15 (LRCK)
- net LRCKB: no longer names the net of IC4.15 (LRCK)
