File: KICAD/STM.kicad_sch (KiCad schematic)
At the start: 1 part, among them IC5 STM32F746BGT6

Commit message: clear
Parts:
- IC5: footprint STM32F746BGT6:QFP50P3000X3000X160-208N -> footprints:STM32F746BGT6
Changed lines of the file:
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@@
 			)
 		)
-		(property "Footprint" "STM32F746BGT6:QFP50P3000X3000X160-208N"
+		(property "Footprint" "footprints:STM32F746BGT6"
 			(at 204.47 158.42 0)
 			(hide yes)

Commit message: presque rien
Connections:
- net AMP_MUTE: no longer names the net of IC5.54 (PA5)
- net AMP_SD: no longer names the net of IC5.53 (PA4)
- net DAC_DIN: no longer names the net of IC5.2 (PE3)
- net JACK_DET: no longer names the net of IC5.45 (PA2)
- net SAI1_FS_A/LRCK: no longer names the net of IC5.3 (PE4)
- net SAI1_MCLK_A/SCKI: no longer names the net of IC5.1 (PE2)
- net SAI1_SCK_A/BCK: no longer names the net of IC5.4 (PE5)
- net SAI1_SD_A/DOUT: no longer names the net of IC5.5 (PE6)
- net USART_RX: no longer names the net of IC5.144 (PA10)
- net USART_TX: no longer names the net of IC5.143 (PA9)
Changed lines of the file:
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@@
 	(generator_version "10.0")
 	(paper "A3")
-	(wire
-		(pts
-			(xy 48.26 76.2) (xy 63.5 76.2)
-		)
-		(stroke
-			(width 0)
-			(type default)
-		)
-	)
-	(wire
-		(pts
-			(xy 48.26 83.82) (xy 63.5 83.82)
-		)
-		(stroke
-			(width 0)
-			(type default)
-		)
-	)
-	(wire
-		(pts
-			(xy 208.28 104.14) (xy 219.71 104.14)
-		)
-		(stroke
-			(width 0)
-			(type default)
-		)
-	)
-	(wire
-		(pts
-			(xy 208.28 106.68) (xy 219.71 106.68)
-		)
-		(stroke
-			(width 0)
-			(type default)
-		)
-	)
-	(wire
-		(pts
-			(xy 48.26 81.28) (xy 63.5 81.28)
-		)
-		(stroke
-			(width 0)
-			(type default)
-		)
-	)
-	(wire
-		(pts
-			(xy 48.26 73.66) (xy 63.5 73.66)
-		)
-		(stroke
-			(width 0)
-			(type default)
-		)
-	)
-	(wire
-		(pts
-			(xy 48.26 78.74) (xy 63.5 78.74)
-		)
-		(stroke
-			(width 0)
-			(type default)
-		)
-	)
-	(hierarchical_label "USART_TX"
-		(shape input)
-		(at 219.71 106.68 0)
-		(effects
-			(font
-				(size 1.27 1.27)
-			)
-			(justify left)
-		)
-	)
-	(hierarchical_label "SAI1_FS_A{slash}LRCK"
-		(shape input)
-		(at 48.26 78.74 180)
-		(effects
-			(font
-				(size 1.27 1.27)
-			)
-			(justify right)
-		)
-	)
-	(hierarchical_label "SAI1_SCK_A{slash}BCK"
-		(shape input)
-		(at 48.26 81.28 180)
-		(effects
-			(font
-				(size 1.27 1.27)
-			)
-			(justify right)
-		)
-	)
-	(hierarchical_label "SAI1_MCLK_A{slash}SCKI"
-		(shape input)
-		(at 48.26 73.66 180)
-		(effects
-			(font
-				(size 1.27 1.27)
-			)
-			(justify right)
-		)
-	)
-	(hierarchical_label "USART_RX"
-		(shape input)
-		(at 219.71 104.14 0)
-		(effects
-			(font
-				(size 1.27 1.27)
-			)
-			(justify left)
-		)
-	)
-	(hierarchical_label "DAC_DIN"
-		(shape input)
-		(at 48.26 76.2 180)
-		(effects
-			(font
-				(size 1.27 1.27)
-			)
-			(justify right)
-		)
-	)
-	(hierarchical_label "SAI1_SD_A{slash}DOUT"
-		(shape input)
-		(at 48.26 83.82 180)
-		(effects
-			(font
-				(size 1.27 1.27)
-			)
-			(justify right)
-		)
-	)
-	(hierarchical_label "AMP_SD"
-		(shape input)
-		(at 71.12 220.98 270)
-		(effects
-			(font
-				(size 1.27 1.27)
-			)
-			(justify right)
-		)
-	)
-	(hierarchical_label "AMP_MUTE"
-		(shape input)
-		(at 73.66 220.98 270)
-		(effects
-			(font
-				(size 1.27 1.27)
-			)
-			(justify right)
-		)
-	)
-	(hierarchical_label "JACK_DET"
-		(shape input)
-		(at 63.5 185.42 180)
-		(effects
-			(font
-				(size 1.27 1.27)
-			)
-			(justify right)
-		)
-	)
 	(symbol
 		(lib_id "STM32F746BGT6:STM32F746BGT6")
