File: KICAD/STM.kicad_sch (KiCad schematic)
At the start: 1 part, among them IC5 STM32F746BGT6

Commit message: mise en forme globale
Connections:
- net DAC_DIN renamed DIN
- net SAI1_FS_A/LRCK renamed LRCK
- net SAI1_MCLK_A/SCKI renamed SCKI
- net SAI1_SCK_A/BCK renamed BCK
- net SAI1_SD_A/DOUT renamed DOUT
Changed lines of the file:
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@@
 		)
 	)
-	(hierarchical_label "SAI1_FS_A{slash}LRCK"
+	(hierarchical_label "LRCK"
 		(shape input)
 		(at 48.26 78.74 180)
@@
 		)
 	)
-	(hierarchical_label "SAI1_SCK_A{slash}BCK"
+	(hierarchical_label "BCK"
 		(shape input)
 		(at 48.26 81.28 180)
@@
 		)
 	)
-	(hierarchical_label "SAI1_MCLK_A{slash}SCKI"
+	(hierarchical_label "SCKI"
 		(shape input)
 		(at 48.26 73.66 180)
@@
 		)
 	)
-	(hierarchical_label "DAC_DIN"
+	(hierarchical_label "DIN"
 		(shape input)
 		(at 48.26 76.2 180)
@@
 		)
 	)
-	(hierarchical_label "SAI1_SD_A{slash}DOUT"
+	(hierarchical_label "DOUT"
 		(shape input)
 		(at 48.26 83.82 180)

Commit message: interface HM
Parts:
- removed IC5: STM32F746BGT6, footprints:STM32F746BGT6, symbol STM32F746BGT6:STM32F746BGT6
- added U4: STM32F446RETx, Package_QFP:LQFP-64_10x10mm_P0.5mm, symbol MCU_ST_STM32F4:STM32F446RETx
Connections:
- new net: U4.18 (VSS), U4.31 (VSS), U4.47 (VSS), U4.63 (VSS)
