File: KICAD/bluetooth.kicad_sch (KiCad schematic)
At the start: 4 parts, among them U1 FSC-BT1026E

Commit message: clear
Parts:
- U1: footprint Bluetooth:FSC-BT1026x -> footprints:FSC-BT1026x
Changed lines of the file:
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@@
 			)
 		)
-		(property "Footprint" "Bluetooth:FSC-BT1026x"
+		(property "Footprint" "footprints:FSC-BT1026x"
 			(at 148.59 48.26 0)
 			(hide yes)

Commit message: presque rien
Parts:
- removed C49: 100n, symbol Device:C_Small
- removed R17: 10 k, symbol Device:R_Small
- added C33, C35: 2.2uF, symbol Device:C_Small
- C36: value 10u -> 2.2uF
Connections:
- net +3.3V: no longer C36.1, U1.34 (SYS_CTRL), U1.36 (VDD_IO)
- net GND: now also C33.2, C35.2; no longer U1.46 (AUDIO_HPR_N), U1.48 (AUDIO_HPL_N)
- net BT_RST: now reaches U1.8 (RESET)
- net BT_MUTE: now reaches U1.16 (BT_RTS/Pl02)
- net at U1.31 (VDD_USB/3.3V_OUT): now also C36.1, U1.36 (VDD_IO), C35.1
- net at U1.35 (1.8V_OUT): now also C33.1
- net I2S_BT_SCK: now reaches U1.4 (PCM_CLK/PI016)
- net I2S_BT_SD: now reaches U1.6 (PCM_OUT/PI018)
- net I2S_BT_WS: now reaches U1.7 (PCM_SYNC/PIO17)
- net AUDIO_HPL_P: no longer names the net of U1.49 (AUDIO_HPL_P)
- net AUDIO_HPR_P: no longer names the net of U1.47 (AUDIO_HPR_P)
- net USART_RX renamed BT_RX
- net USART_TX renamed BT_TX
- new net BT_EN: U1.34 (SYS_CTRL)
- no-connect marks 2 -> 0
