File: KICAD/bluetooth.kicad_sch (KiCad schematic)
At the start: 4 parts, among them U1 FSC-BT1026E

Commit message: mise en forme globale
Connections:
- net +3.3V: no longer C36.1, C49.1, R17.2, U1.33 (VBAT_IN), U1.34 (SYS_CTRL)
- new net +3V3: C36.1, C49.1, R17.2, U1.33 (VBAT_IN), U1.34 (SYS_CTRL)
Changed lines of the file:
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@@
 			)
 		)
-		(property "Value" "+3.3V"
-			(at 123.19 17.78 0)
-			(show_name no)
-			(do_not_autoplace no)
-			(effects
-				(font
-					(size 1.27 1.27)
-				)
+		(property "Value" "+3V3"
+			(at 125.73 21.5899 0)
+			(show_name no)
+			(do_not_autoplace no)
+			(effects
+				(font
+					(size 1.27 1.27)
+				)
+				(justify left)
 			)
 		)
@@
 			)
 		)
-		(property "Value" "+3.3V"
+		(property "Value" "+3V3"
 			(at 80.01 49.53 90)
 			(show_name no)

Commit message: on ne sair jamais
Connections:
- net +3.3V is gone; now on net +3V3: U1.36 (VDD_IO)

Commit message: interface HM
Connections:
- net USART_RX renamed BT_RX
- net USART_TX renamed BT_TX
Changed lines of the file:
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@@
 		)
 	)
-	(hierarchical_label "USART_TX"
+	(hierarchical_label "BT_TX"
 		(shape input)
 		(at 99.06 67.31 180)
@@
 		)
 	)
-	(hierarchical_label "USART_RX"
+	(hierarchical_label "BT_RX"
 		(shape input)
 		(at 99.06 64.77 180)
