File: KICAD/projet_2A.kicad_sch (KiCad schematic)
At the start: 3 parts, among them J1 AudioJack3_Ground_Switch

Commit message: presque rien
Parts:
- removed R24, R25: 1k, symbol Device:R_Small
Connections:
- net Bluetooth/AUDIO_HPL_P: no longer names the net of J1.TN
- net Bluetooth/AUDIO_HPR_P: no longer names the net of J1.RN
- net GND: no longer names the net of J1.S
- net JACK_DET: no longer names the net of J1.G
- net R/VINR: no longer names the net of J1.R
- net T/VINL: no longer names the net of J1.T
- no-connect marks 1 -> 0
Other:
- sheet ADC_PCM1808 ports: added none; removed BCK/SAI1_SCK_A, DOUT/SAI1_SD_A, LRCK/SAI1_FS_A, R/VINR, SCKI/SAI1_MCLK_A, T/VINL
- sheet Bluetooth ports: added none; removed AUDIO_HPL_P, AUDIO_HPR_P, USART_RX, USART_TX
- sheet DAC_PCM5102A ports: added none; removed BCKA, BCKB, DIN/SAI1_SD_A, DIN/SAI1_SD_B, LRCKA, LRCKB, SPK_L, SPK_R, SUB_L, SUB_R
- sheet STM ports: added none; removed AMP_MUTE, AMP_SD, DAC_DIN, JACK_DET, SAI1_FS_A/LRCK, SAI1_MCLK_A/SCKI, SAI1_SCK_A/BCK, SAI1_SD_A/DOUT, USART_RX, USART_TX
- sheet TPA3116D2 ports: added none; removed IN_N_LEFT, IN_N_RIGHT, IN_N_SUB, IN_P_LEFT, IN_P_RIGHT, IN_P_SUB, MUTE_LR, MUTE_SUB, OUT_N_LEFT, OUT_N_RIGHT, OUT_N_SUB, OUT_P_LEFT, OUT_P_RIGHT, OUT_P_SUB, SD_LR, SD_SUB
